File: fmba/KiCadVcu/vcu-pi/vcu-pi.sch (KiCad schematic (older format))
At the start: 57 parts, among them P1 CONN_01X08, P2 CONN_02X12, P3 CONN_02X20, P4 CONN_01X12, U1 THN_15-2411WI_, U10 PC817, U2 NCV1124, U3 NCV1124, U4 PC817, U5 PC817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

Commit message: kicad rescue changes
Parts:
- U1: symbol thn_15-2411wi_:THN_15-2411WI_ -> vcu-pi-rescue:THN_15-2411WI_-thn_15-2411wi_
- U2, U3: symbol ncv1124:NCV1124 -> vcu-pi-rescue:NCV1124-ncv1124
Changed lines of the file:
@@
 EESchema Schematic File Version 4
 LIBS:vcu-pi-cache
-EELAYER 29 0
+EELAYER 26 0
 EELAYER END
 $Descr A4 11693 8268
@@
 $EndComp
 $Comp
-L ncv1124:NCV1124 U3
+L vcu-pi-rescue:NCV1124-ncv1124 U3
 U 1 1 5C87C5B2
 P 2250 5250
@@
 $EndComp
 $Comp
-L thn_15-2411wi_:THN_15-2411WI_ U1
+L vcu-pi-rescue:THN_15-2411WI_-thn_15-2411wi_ U1
 U 1 1 5C87C7FC
 P 1800 1600
@@
 $EndComp
 $Comp
-L ncv1124:NCV1124 U2
+L vcu-pi-rescue:NCV1124-ncv1124 U2
 U 1 1 5C883995
 P 2200 6850
